Commit message: arm FINALLY MOVES with prefix ur5_

File: ur_gazebo/inc/urdf/ur.xacro (robot description, xacro)
@@ -44,5 +44,5 @@
   <!-- Instantiate the Gazebo robot and pass it all the required arguments. -->
   <xacro:ur_robot_gazebo
-    prefix=""
+    prefix="ur5_"
     joint_limits_parameters_file="$(arg joint_limit_params)"
     kinematics_parameters_file="$(arg kinematics_params)"
@@ -64,10 +64,10 @@
   <joint name="world_joint" type="fixed">
     <parent link="world"/>
-    <child link="base_link"/>
+    <child link="ur5_base_link"/>
     <origin xyz="0 0 0" rpy="0 0 0"/>
   </joint>
   <link name="tool0_controller"/>
   <joint name="tool_controller_fake_joint" type="fixed">
-    <parent link="tool0"/>
+    <parent link="ur5_tool0"/>
     <child link="tool0_controller"/>
     <origin xyz="0 0 0" rpy="0 0 0"/>
