Commit message: impakt.launch has includes which launches one from two robots, other is commented"

File: impakt_robot.urdf.xacro (robot description, xacro)
@@ -2,5 +2,5 @@
 <robot xmlns:xacro="http://www.ros.org/wiki/xacro" name="impakt_robot">
     <xacro:include filename="$(find neo_simulation)/robots/mp_500/mp_500.urdf.xacro"/>
-    <origin xyz="2 2 0"/>
+    <!-- <origin xyz="2 2 0"/>
     <xacro:arg name="robot_model" default="ur5"/>
     <xacro:arg name="joint_limit_params" default="$(find ur_description)/config/ur5/joint_limits.yaml"/>
@@ -28,4 +28,4 @@
         <child link="ur5_base_link"/>
         <origin xyz="0 0 0.5" rpy="0 0 90"/>
-    </joint>
+    </joint> -->
 </robot>

Commit message: reference impakt_robot.urdf.xacro

File: impakt_robot.urdf.xacro (robot description, xacro)
@@ -1,31 +1,75 @@
 <?xml version="1.0"?>
-<robot xmlns:xacro="http://www.ros.org/wiki/xacro" name="impakt_robot">
-    <xacro:include filename="$(find neo_simulation)/robots/mp_500/mp_500.urdf.xacro"/>
-    <!-- <origin xyz="2 2 0"/>
-    <xacro:arg name="robot_model" default="ur5"/>
-    <xacro:arg name="joint_limit_params" default="$(find ur_description)/config/ur5/joint_limits.yaml"/>
-    <xacro:arg name="kinematics_params" default="$(find ur_description)/config/ur5/default_kinematics.yaml"/>
-    <xacro:arg name="physical_params" default="$(find ur_description)/config/ur5/physical_parameters.yaml"/>
-    <xacro:arg name="visual_params" default="$(find ur_description)/config/ur5/visual_parameters.yaml"/>
-    <xacro:arg name="transmission_hw_interface" default="hardware_interface/EffortJointInterface"/>
-    <xacro:arg name="safety_limits" default="false"/>
-    <xacro:arg name="safety_pos_margin" default="0.15"/>
-    <xacro:arg name="safety_k_position" default="20"/>
-    <xacro:include filename="$(find ur_gazebo)/urdf/ur_macro.xacro"/>
-    <xacro:ur_robot_gazebo
-        prefix="ur5_"
-        joint_limits_parameters_file="$(arg joint_limit_params)"
-        kinematics_parameters_file="$(arg kinematics_params)"
-        physical_parameters_file="$(arg physical_params)"
-        visual_parameters_file="$(arg visual_params)"
-        transmission_hw_interface="$(arg transmission_hw_interface)"
-        safety_limits="$(arg safety_limits)"
-        safety_pos_margin="$(arg safety_pos_margin)"
-        safety_k_position="$(arg safety_k_position)"
-    />
-    <joint name="world_joint" type="fixed">
-        <parent link="base_link"/>
-        <child link="ur5_base_link"/>
-        <origin xyz="0 0 0.5" rpy="0 0 90"/>
-    </joint> -->
+<robot xmlns:xacro="http://wiki.ros.org/xacro" name="$(arg robot_model)_robot">
+  <!--
+    This is a top-level xacro instantiating the Gazebo-specific version of the
+    'ur_robot' macro (ie: 'ur_robot_gazebo') and passing it values for all its
+    required arguments.
+    This file should be considered the Gazebo-specific variant of the file
+    with the same name in the ur_description package. It accepts the same
+    arguments, but instead of configuring everything for a real robot, will
+    generate a Gazebo-compatible URDF with a ros_control hardware_interface
+    attached to it.
+    Only use this top-level xacro if you plan on spawning the robot in Gazebo
+    'by itself', without any gripper or any other geometry attached.
+    If you need to attach an end-effector, camera or need to integrate the
+    robot into a larger workcell and want to spawn that as a single entity in
+    Gazebo, DO NOT EDIT THIS FILE.
+    Instead: create a new top-level xacro, give it a proper name, include the
+    required '.xacro' files, instantiate the models (ie: call the macros) and
+    connect everything by adding the appropriate joints.
+  -->
+  <!--
+    Import main macro.
+    NOTE: this imports the Gazebo-wrapper main macro, NOT the regular
+          xacro macro (which is hosted by ur_description).
+  -->
+  <xacro:include filename="$(find ur_gazebo)/urdf/ur_macro.xacro"/>
+  <!--Declare arguments -->
+  <xacro:arg name="joint_limit_params" default=""/>
+  <xacro:arg name="physical_params" default=""/>
+  <xacro:arg name="kinematics_params" default=""/>
+  <xacro:arg name="visual_params" default=""/>
+  <!--
+    legal values:
+      - hardware_interface/PositionJointInterface
+      - hardware_interface/VelocityJointInterface
+      - hardware_interface/EffortJointInterface
+    NOTE: this value must correspond to the controller configured in the
+          controller .yaml files in the 'config' directory.
+  -->
+  <xacro:arg name="transmission_hw_interface" default="hardware_interface/EffortJointInterface"/>
+  <xacro:arg name="safety_limits" default="false"/>
+  <xacro:arg name="safety_pos_margin" default="0.15"/>
+  <xacro:arg name="safety_k_position" default="20"/>
+  <!-- Instantiate the Gazebo robot and pass it all the required arguments. -->
+  <xacro:ur_robot_gazebo
+    prefix="ur5_"
+    joint_limits_parameters_file="$(arg joint_limit_params)"
+    kinematics_parameters_file="$(arg kinematics_params)"
+    physical_parameters_file="$(arg physical_params)"
+    visual_parameters_file="$(arg visual_params)"
+    transmission_hw_interface="$(arg transmission_hw_interface)"
+    safety_limits="$(arg safety_limits)"
+    safety_pos_margin="$(arg safety_pos_margin)"
+    safety_k_position="$(arg safety_k_position)"
+  />
+  <!--
+    Attach the Gazebo model to Gazebo's world frame.
+    Note: if you're looking to integrate a UR into a larger scene and need
+    to add EEFs or other parts, DO NOT change this file or the 'world' link
+    here. Create a NEW xacro instead and decide whether you need to add
+    a 'world' link there.
+  -->
+  <link name="world"/>
+  <joint name="world_joint" type="fixed">
+    <parent link="world"/>
+    <child link="ur5_base_link"/>
+    <origin xyz="0 0 0" rpy="0 0 0"/>
+  </joint>
+  <link name="tool0_controller"/>
+  <joint name="tool_controller_fake_joint" type="fixed">
+    <parent link="ur5_tool0"/>
+    <child link="tool0_controller"/>
+    <origin xyz="0 0 0" rpy="0 0 0"/>
+  </joint>
 </robot>

Commit message: ITS ALIVE

File: impakt_robot.urdf.xacro (robot description, xacro)
@@ -1,4 +1,4 @@
 <?xml version="1.0"?>
-<robot xmlns:xacro="http://wiki.ros.org/xacro" name="$(arg robot_model)_robot">
+<robot xmlns:xacro="http://wiki.ros.org/xacro" name="impakt_robot">
   <!--
     This is a top-level xacro instantiating the Gazebo-specific version of the
@@ -24,4 +24,6 @@
           xacro macro (which is hosted by ur_description).
   -->
+  <xacro:include filename="$(find neo_simulation)/robots/mp_500/mp_500.urdf.xacro"/>
+  <origin xyz="2 2 0"/>
   <xacro:include filename="$(find ur_gazebo)/urdf/ur_macro.xacro"/>
   <!--Declare arguments -->
@@ -61,9 +63,8 @@
     a 'world' link there.
   -->
-  <link name="world"/>
   <joint name="world_joint" type="fixed">
-    <parent link="world"/>
+    <parent link="base_link"/>
     <child link="ur5_base_link"/>
-    <origin xyz="0 0 0" rpy="0 0 0"/>
+    <origin xyz="0 0 0.5" rpy="0 0 90"/>
   </joint>
   <link name="tool0_controller"/>

Commit message: change arm position

File: impakt_robot.urdf.xacro (robot description, xacro)
@@ -66,5 +66,5 @@
     <parent link="base_link"/>
     <child link="ur5_base_link"/>
-    <origin xyz="0 0 0.5" rpy="0 0 90"/>
+    <origin xyz="-0.2 0 0.34" rpy="0 0 185"/>
   </joint>
   <link name="tool0_controller"/>

Commit message: add boxes

File: impakt_robot.urdf.xacro (robot description, xacro)
@@ -24,5 +24,5 @@
           xacro macro (which is hosted by ur_description).
   -->
-  <xacro:include filename="$(find neo_simulation)/robots/mp_500/mp_500.urdf.xacro"/>
+  <xacro:include filename="$(find impakt-robot)/neo_simulation/robots/mp_500/mp_500.urdf.xacro"/>
   <origin xyz="2 2 0"/>
   <xacro:include filename="$(find impakt-robot)/ur_macro.xacro"/>
@@ -64,7 +64,7 @@
   -->
   <joint name="world_joint" type="fixed">
-    <parent link="base_link"/>
-    <child link="ur5_base_link"/>
-    <origin xyz="-0.2 0 0.34" rpy="0 0 185"/>
+      <parent link="above_body_platform_link"/>
+      <child link="ur5_base_link"/>
+      <origin xyz="0.05 0 0.075" rpy="0 0 0"/>
   </joint>
   <link name="tool0_controller"/>
